Commit message: moveit config initial setup

File: ur10_description/urdf/mech/end_effector.urdf.xacro (robot description, xacro)
@@ -7,7 +7,7 @@
     <link name="${prefix}ee_link">
       <visual>
-        <origin xyz="0 0 0" rpy="0 0 0"/>
+        <origin xyz="0 0 0" rpy="-1.5708 0 0"/>
         <geometry>
-          <mesh filename="package://ur10_description/meshes/ee/collision/mock-up-end-effector.stl" scale="0.001 0.001 0.001"/>
+          <mesh filename="package://ur10_description/meshes/ee/visual/mock-up-end-effector.dae" scale="1 1 1"/>
         </geometry>
       </visual>
