Commit message: testing

File: ur10_description/urdf/robots/custom_ur10.urdf.xacro (robot description, xacro)
@@ -1,4 +1,5 @@
 <?xml version="1.0"?>
 <robot xmlns:xacro="http://www.ros.org/wiki/xacro" name="ur10_with_custom_ee">
+  <xacro:arg name="use_gazebo" default="false" />
   <link name="world"/>
   <xacro:property name="robot_prefix" value="" />
@@ -21,3 +22,11 @@
   <xacro:include filename="$(find ur10_description)/urdf/mech/end_effector.urdf.xacro" />
   <xacro:end_effector parent_link_name="${robot_prefix}tool0" prefix="custom_"/>
-</robot>
+  <xacro:include filename="$(find ur10_description)/urdf/ur10.gazebo.xacro" />
+  <xacro:ur10_gazebo_ros2_control_plugin use_gazebo="$(arg use_gazebo)" />
+  <xacro:include filename="$(find ur10_moveit_config)/config/ur10_with_custom_ee.ros2_control.xacro" />
+  <xacro:ur10_with_custom_ee_ros2_control
+      name="UR10"
+      initial_positions_file="$(find ur10_moveit_config)/config/initial_positions.yaml"
+      use_gazebo="$(arg use_gazebo)"
+      />
+  </robot>

File: ur10_moveit_config/config/ur10_with_custom_ee.ros2_control.xacro (robot description, xacro)
@@ -1,70 +1,56 @@
 <?xml version="1.0"?>
 <robot xmlns:xacro="http://www.ros.org/wiki/xacro">
-    <xacro:macro name="ur10_with_custom_ee_ros2_control" params="name initial_positions_file">
+    <xacro:macro name="ur10_with_custom_ee_ros2_control" params="name initial_positions_file use_gazebo">
         <xacro:property name="initial_positions" value="${xacro.load_yaml(initial_positions_file)['initial_positions']}"/>
         <ros2_control name="${name}" type="system">
             <hardware>
-                <!-- By default, set up controllers for simulation. This won't work on real hardware -->
-                <plugin>mock_components/GenericSystem</plugin>
+                <xacro:if value="${use_gazebo}">
+                    <plugin>gz_ros2_control/GazeboSimSystem</plugin>
+                </xacro:if>
+                <xacro:unless value="${use_gazebo}">
+                    <plugin>mock_components/GenericSystem</plugin>
+                </xacro:unless>
             </hardware>
             <joint name="shoulder_pan_joint">
                 <command_interface name="position"/>
-                <command_interface name="velocity"/>
-                <command_interface name="effort"/>
                 <state_interface name="position">
                   <param name="initial_value">${initial_positions['shoulder_pan_joint']}</param>
                 </state_interface>
                 <state_interface name="velocity"/>
-                <state_interface name="effort"/>
             </joint>
             <joint name="shoulder_lift_joint">
                 <command_interface name="position"/>
-                <command_interface name="velocity"/>
-                <command_interface name="effort"/>
                 <state_interface name="position">
                   <param name="initial_value">${initial_positions['shoulder_lift_joint']}</param>
                 </state_interface>
                 <state_interface name="velocity"/>
-                <state_interface name="effort"/>
             </joint>
             <joint name="elbow_joint">
                 <command_interface name="position"/>
-                <command_interface name="velocity"/>
-                <command_interface name="effort"/>
                 <state_interface name="position">
                   <param name="initial_value">${initial_positions['elbow_joint']}</param>
                 </state_interface>
                 <state_interface name="velocity"/>
-                <state_interface name="effort"/>
             </joint>
             <joint name="wrist_1_joint">
                 <command_interface name="position"/>
-                <command_interface name="velocity"/>
-                <command_interface name="effort"/>
                 <state_interface name="position">
                   <param name="initial_value">${initial_positions['wrist_1_joint']}</param>
                 </state_interface>
                 <state_interface name="velocity"/>
-                <state_interface name="effort"/>
             </joint>
             <joint name="wrist_2_joint">
                 <command_interface name="position"/>
-                <command_interface name="velocity"/>
-                <command_interface name="effort"/>
                 <state_interface name="position">
                   <param name="initial_value">${initial_positions['wrist_2_joint']}</param>
                 </state_interface>
                 <state_interface name="velocity"/>
-                <state_interface name="effort"/>
             </joint>
             <joint name="wrist_3_joint">
                 <command_interface name="position"/>
-                <command_interface name="velocity"/>
-                <command_interface name="effort"/>
                 <state_interface name="position">
                   <param name="initial_value">${initial_positions['wrist_3_joint']}</param>
                 </state_interface>
                 <state_interface name="velocity"/>
-                <state_interface name="effort"/>
             </joint>
         </ros2_control>
