Commit message: Defined Tool Center Point for weld kinematics
- Added "custom_tcp_link"  and a fixed joint with Z-offset inside the end-effector Xacro macro to represent the physical tip
- Updated SRDF "arm" planning group to extend kinematic chain from "base_link" to "custom_tcp_link"
- Fixed the reversed group definitions in the SRDF "<end_effector>" tag to prevent MoveIt hierarchy confusion

File: src/ur10_description/urdf/mech/end_effector.urdf.xacro (robot description, xacro)
@@ -32,4 +32,10 @@
         <origin xyz="0 0 0" rpy="0 0 ${pi}"/>
     </joint>
+    <link name="${prefix}tcp_link"/>
+    <joint name="${prefix}tcp_joint" type="fixed">
+      <origin xyz="0 0 0.15" rpy="0 0 0"/>
+      <parent link="${parent_link_name}"/>
+      <child link="${prefix}tcp_link"/>
+    </joint>
   </xacro:macro>
 </robot>
